Commit message: Added the code for Gazebo Simulation Control

File: description/robot.urdf.xacro (robot description, xacro)
@@ -3,3 +3,5 @@
     <!-- Defines the file for the robot's body [Source 3]-->
     <xacro:include filename="robot_core.xacro"/>
+    <!-- Defines the file for the robot's body [Source 5]-->
+    <xacro:include filename="gazebo_control.xacro"/>
 </robot>

File: description/robot_core.xacro (robot description, xacro)
@@ -1,5 +1,5 @@
 <?xml version="1.0"?>
 <robot xmlns:xacro="http://www.ros.org/wiki/xacro">
-    <!-- Calls the inertial macros to provide inertia [Source 4]-->
+    <!-- 1. Calls the inertial macros to provide inertia [Source 4]-->
     <xacro:include filename="inertial_macros.xacro"/>
     <!-- 2. Defines all the relevant colours of materials [Source 3]-->
@@ -44,4 +44,7 @@
         </xacro:inertial_box>
     </link>
+    <gazebo reference="chassis">
+        <material>Gazebo/White</material>
+    </gazebo>
     <!-- 3C. This is the left wheel, a cylinder with a radius of 5cm and length of 4cm, with an y-offset of 175mm and rotated 270 degrees around the x-axis-->
     <joint name="left_wheel_joint" type="continous">
@@ -67,4 +70,7 @@
         </xacro:inertial_cylinder>
     </link>
+    <gazebo reference="left_wheel">
+        <material>Gazebo/Black</material>
+    </gazebo>
     <!-- 3D. This is the right wheel, a cylinder with a radius of 5cm and length of 4cm, with an y-offset of 175mm and rotated 90 degrees around the x-axis-->
     <joint name="right_wheel_joint" type="continous">
@@ -90,4 +96,7 @@
         </xacro:inertial_cylinder>
     </link>
+    <gazebo reference="right_wheel">
+        <material>Gazebo/Black</material>
+    </gazebo>
     <!-- 3E. This is the caster wheel, a sphere with a radius of 5cm, located at an x-offset of 24cm from the chassis-->
     <joint name="caster_wheel_joint" type="fixed">
@@ -112,3 +121,8 @@
         </xacro:inertial_sphere>
     </link>
+    <gazebo reference="caster_wheel">
+        <material>Gazebo/Black</material>
+        <mu1 value="0.001"/>
+        <mu2 value="0.001"/>
+    </gazebo>
 </robot>

Commit message: Introducing Lidar and Camera

File: description/robot.urdf.xacro (robot description, xacro)
@@ -5,3 +5,7 @@
     <!-- Defines the file for the robot's body [Source 5]-->
     <xacro:include filename="gazebo_control.xacro"/>
+    <!-- Defines the file for the robot's body [Source 11]-->
+    <xacro:include filename="lidar.xacro"/>
+    <!-- Defines the file for the robot's body [Source 14]-->
+    <xacro:include filename="camera.xacro"/>
 </robot>

File: description/robot_core.xacro (robot description, xacro)
@@ -12,4 +12,7 @@
     <material name="blue">
         <color rgba="0.2 0.2 1 1"/>
+    </material>
+    <material name="red">
+        <color rgba="1 0 0 1"/>
     </material>
     <material name="black">
