Commit message: Introducing depth camera, ros2 controls, and edited the configs to increase stability

File: description/depth_camera.xacro (robot description, xacro)
@@ -32,8 +32,8 @@
     </joint>
     <link name="camera_link_optical"> </link>
-    <!-- 2. Gazebo reference for camera_link [Source 12]-->
+    <!-- 2. Gazebo reference for camera_link [Source 15]-->
     <gazebo reference="camera_link">
         <material>Gazebo/Red</material>
-        <sensor name="camera" type="camera">
+        <sensor name="camera" type="depth">
             <pose> 0 0 0 0 0 0 </pose>
             <visualize>true</visualize>
@@ -44,5 +44,5 @@
                     <width>640</width>
                     <height>480</height>
-                    <format>R8G8B8</format>
+                    <format>B8G8R8</format>
                 </image>
                 <clip>
@@ -53,4 +53,6 @@
             <plugin name="camera_controller" filename="libgazebo_ros_camera.so">
                 <frame_name>camera_link_optical</frame_name>
+                <min depth>0.1</min_depth>
+                <max depth>100</max_depth>
             </plugin>
         </sensor>

File: description/gazebo_control.xacro (robot description, xacro)
@@ -1,2 +1,3 @@
+<!--This code has been obtained from source 5-->
 <?xml version="1.0"?>
 <robot xmlns:xacro="http://www.ros.org/wiki/xacro">

File: description/robot.urdf.xacro (robot description, xacro)
@@ -1,11 +1,23 @@
 <?xml version="1.0"?>
 <robot xmlns:xacro="http://www.ros.org/wiki/xacro"  name="robot">
-    <!-- Defines the file for the robot's body [Source 3]-->
+    <!-- 1. Defines the file for the robot's body [Source 3]-->
     <xacro:include filename="robot_core.xacro"/>
-    <!-- Defines the file for the robot's body [Source 5]-->
-    <xacro:include filename="gazebo_control.xacro"/>
-    <!-- Defines the file for the robot's body [Source 11]-->
+    <!-- 2. Defines the file for the robot's control (Note - ONLY ONE CAN BE ACTIVE AT A TIME)-->
+    <!-- 2A. A boolean to determine which controls to use [Source 19]-->
+    <xacro:arg name="use_ros2_control" default="true"/>
+    <!-- 2B. Defines the file for the robot's real-life control using ROS2 [Source 17]-->
+    <xacro:if value="$(arg use_ros2_control)">
+        <xacro:include filename="ros2_control.xacro"/>
+    </xacro:if>
+    <!-- 2C. Defines the file for the robot's simulation control usig Gazebo [Source 5]-->
+    <xacro:unless value="$(arg use_ros2_control)">
+        <xacro:include filename="gazebo_control.xacro"/>
+    </xacro:unless>
+    <!-- 3. Defines the file for the robot's lidar [Source 11]-->
     <xacro:include filename="lidar.xacro"/>
-    <!-- Defines the file for the robot's body [Source 14]-->
+    <!-- 4. Defines the file for the robot's cameras (Note - ONLY ONE CAN BE ACTIVE AT A TIME)-->
+    <!-- 4A. Defines the file for the robot's camera [Source 14]-->
     <xacro:include filename="camera.xacro"/>
+    <!-- 4B. Defines the file for the robot's depth camere [Source 15]-->
+    <!-- <xacro:include filename="depth_camera.xacro"/> -->
 </robot>

File: description/robot_core.xacro (robot description, xacro)
@@ -3,5 +3,20 @@
     <!-- 1. Calls the inertial macros to provide inertia [Source 4]-->
     <xacro:include filename="inertial_macros.xacro"/>
-    <!-- 2. Defines all the relevant colours of materials [Source 3]-->
+    <!-- 2. Defines all the relevant dimensions [Source 19]-->
+    <xacro:property name="chassis_length" value="0.335"/>
+    <xacro:property name="chassis_width" value="0.265"/>
+    <xacro:property name="chassis_height" value="0.138"/>
+    <xacro:property name="chassis_mass" value="1.0"/>
+    <xacro:property name="wheel_radius" value="0.034"/>
+    <xacro:property name="wheel_thickness" value="0.026"/>
+    <xacro:property name="wheel_mass" value="0.05"/>
+    <xacro:property name="wheel_offset_x" value="0.226"/>
+    <xacro:property name="wheel_offset_y" value="0.166"/>
+    <xacro:property name="wheel_offset_z" value="0.01"/>
+    <xacro:property name="caster_wheel_radius" value="0.01"/>
+    <xacro:property name="caster_wheel_mass" value="0.01"/>
+    <xacro:property name="caster_wheel_offset_x" value="0.075"/>
+    <xacro:property name="caster_wheel_offset_z" value="${wheel_offset_z - wheel_radius + caster_wheel_radius}"/>
+    <!-- 3. Defines all the relevant colours of materials [Source 3]-->
     <material name="white">
         <color rgba="1 1 1 1"/>
@@ -19,30 +34,30 @@
         <color rgba="0 0 0 1"/>
     </material>
-    <!-- 3. Defines all the relevant links of the body [Source 3]-->
-    <!-- 3A. This is the base link, located at the centre of the body. All points will be based of this-->
+    <!-- 4. Defines all the relevant links of the body [Source 3 and 19]-->
+    <!-- 4A. This is the base link, located at the centre of the body. All points will be based of this-->
     <link name="base_link">
     </link>
-    <!-- 3B. This is the chassis, a box with a size of 30cm x 30cm x 15cm, located at the origin of the base link with an x-offset of 15cm and z-offset of 7.5cm-->
+    <!-- 4B. This is the chassis, a box with a size of 30cm x 30cm x 15cm, located at the origin of the base link with an x-offset of 15cm and z-offset of 7.5cm-->
     <joint name="chassis_joint" type="fixed">
         <parent link="base_link"/>
         <child link="chassis"/>
-        <origin xyz="-0.1 0 0" rpy="0 0 0"/>
+        <origin xyz="${-wheel_offset_x} 0 ${-wheel_offset_z}"/>
     </joint>
     <link name="chassis">
         <visual>
-            <origin xyz="0.15 0 0.075" rpy="0 0 0"/>
+            <origin xyz="${chassis_length/2} 0 ${chassis_height/2}"/>
             <geometry>
-                <box size="0.3 0.3 0.15"/>
+                <box size="${chassis_length} ${chassis_width} ${chassis_height}"/>
             </geometry>
             <material name="white"/>
         </visual>
         <collision>
-            <origin xyz="0.15 0 0.075" rpy="0 0 0"/>
+            <origin xyz="${chassis_length/2} 0 ${chassis_height/2}"/>
             <geometry>
-                <box size="0.3 0.3 0.15"/>
+                <box size="${chassis_length} ${chassis_width} ${chassis_height}"/>
             </geometry>
         </collision>
-        <xacro:inertial_box mass="0.5" x="0.3" y="0.3" z="0.15"/>
-            <origin xyz="0.15 0 0.075" rpy="0 0 0"/>
+        <xacro:inertial_box mass="0.5" x="${chassis_length}" y="${chassis_width}" z="${chassis_height}">
+            <origin xyz="${chassis_length/2} 0 ${chassis_height/2}" rpy="0 0 0"/>
         </xacro:inertial_box>
     </link>
@@ -54,5 +69,5 @@
         <parent link="base_link"/>
         <child link="left_wheel"/>
-        <origin xyz="0 0.175 0" rpy="-${pi/2} 0 0"/>
+        <origin xyz="0 ${wheel_offset_y} 0" rpy="-${pi/2} 0 0" />
         <axis xyz="0 0 1"/>
     </joint>
@@ -60,5 +75,5 @@
         <visual>
             <geometry>
-                <cylinder radius="0.05" length="0.04"/>
+                <cylinder radius="${wheel_radius}" length="${wheel_thickness}"/>
             </geometry>
             <material name="black"/>
@@ -66,8 +81,8 @@
         <collision>
             <geometry>
-                <cylinder radius="0.05" length="0.04"/>
+                <sphere radius="${wheel_radius}"/>
             </geometry>
         </collision>
-        <xacro:inertial_cylinder mass="0.1" length="0.04" radius="0.05"/>
+        <xacro:inertial_cylinder mass="${wheel_mass}" length="${wheel_thickness}" radius="${wheel_radius}">
             <origin xyz="0 0 0" rpy="-${pi/2} 0 0"/>
         </xacro:inertial_cylinder>
@@ -80,5 +95,5 @@
         <parent link="base_link"/>
         <child link="right_wheel"/>
-        <origin xyz="0 -0.175 0" rpy="${pi/2} 0 0"/>
+        <origin xyz="0 ${-wheel_offset_y} 0" rpy="${pi/2} 0 0" />
         <axis xyz="0 0 -1"/>
     </joint>
@@ -86,5 +101,5 @@
         <visual>
             <geometry>
-                <cylinder radius="0.05" length="0.04"/>
+                <cylinder radius="${wheel_radius}" length="${wheel_thickness}"/>
             </geometry>
             <material name="black"/>
@@ -92,8 +107,8 @@
         <collision>
             <geometry>
-                <cylinder radius="0.05" length="0.04"/>
+                <sphere radius="${wheel_radius}"/>
             </geometry>
         </collision>
-        <xacro:inertial_cylinder mass="0.1" length="0.04" radius="0.05"/>
+        <xacro:inertial_cylinder mass="${wheel_mass}" length="${wheel_thickness}" radius="${wheel_radius}">
             <origin xyz="0 0 0" rpy="-${pi/2} 0 0"/>
         </xacro:inertial_cylinder>
@@ -106,10 +121,10 @@
         <parent link="chassis"/>
         <child link="caster_wheel"/>
-        <origin xyz="0.24 0 0"/>
+        <origin xyz="${caster_wheel_offset_x} 0 ${caster_wheel_offset_z}"/>
     </joint>
     <link name="caster_wheel">
         <visual>
             <geometry>
-                <sphere radius="0.05"/>
+                <sphere radius="${caster_wheel_radius}"/>
             </geometry>
             <material name="black"/>
@@ -117,8 +132,8 @@
         <collision>
             <geometry>
-                <sphere radius="0.05"/>
+                <sphere radius="${caster_wheel_radius}"/>
             </geometry>
         </collision>
-        <xacro:inertial_sphere mass="0.1" radius="0.05"/>
+         <xacro:inertial_sphere mass="${caster_wheel_mass}" radius="${caster_wheel_radius}">
             <origin xyz="0 0 0" rpy ="0 0 0"/>
         </xacro:inertial_sphere>
