Commit message: Introducing ability to toggle between simulation and real world modes

File: description/gazebo_control.xacro (robot description, xacro)
@@ -1,4 +1,4 @@
+<?xml version="1.0"?>
 <!--This code has been obtained from source 5-->
-<?xml version="1.0"?>
 <robot xmlns:xacro="http://www.ros.org/wiki/xacro">
     <!-- 1. Introduces the gazebo (simulation) controls-->

File: description/inertial_macros.xacro (robot description, xacro)
@@ -1,4 +1,4 @@
+<?xml version="1.0"?>
 <!--This code has been obtained from source 4-->
-<?xml version="1.0"?>
 <robot xmlns:xacro="http://www.ros.org/wiki/xacro" >
     <!-- Specify some standard inertial calculations https://en.wikipedia.org/wiki/List_of_moments_of_inertia -->

File: description/robot.urdf.xacro (robot description, xacro)
@@ -6,4 +6,6 @@
     <!-- 2A. A boolean to determine which controls to use [Source 19]-->
     <xacro:arg name="use_ros2_control" default="true"/>
+    <!-- Boolean to toggle simulation mode and real world mode [Source 20]-->
+    <xacro:arg name="sim_mode" default="false"/>
     <!-- 2B. Defines the file for the robot's real-life control using ROS2 [Source 17]-->
     <xacro:if value="$(arg use_ros2_control)">

File: description/ros2_control.xacro (robot description, xacro)
@@ -1,31 +1,66 @@
+<?xml version="1.0"?>
 <!--This code has been obtained from source 17-->
-<?xml version="1.0"?>
 <robot xmlns:xacro="http://www.ros.org/wiki/xacro">
     <!-- 1. Introduces the hardware control-->
-    <ros2_control name="GazeboSystem" type="system">
-        <hardware>
-            <plugin>gazebo_ros2_control/GazeboSystem</plugin>
-        </hardware>
-        <joint name = "left_wheel_joint">
-            <command_interface name = "velocity">
-                <param name="min">-10.0</param>
-                <param name="max">10.0</param>
-            </command_interface>
-            <state_interface name = "velocity"/>
-            <state_interface name = "position"/>
-        </joint>
-        <joint name = "right_wheel_joint">
-            <command_interface name = "velocity">
-                <param name="min">-10.0</param>
-                <param name="max">10.0</param>
-            </command_interface>
-            <state_interface name = "velocity"/>
-            <state_interface name = "position"/>
-        </joint>
-    </ros2_control>
+    <!-- 1A. Real world mode-->
+    <xacro:unless value="$(arg sim_mode)">
+        <ros2_control name="RealRobot" type="system">
+            <hardware>
+                <plugin>diffdrive_arduino/DiffDriveArduino</plugin>
+                <param name="left_wheel_name"></param>
+                <param name="right_wheel_name"></param>
+                <param name="loop_rate"></param>
+                <param name="device"></param>
+                <param name="baud_rate"></param>
+                <param name="timeout"></param>
+                <param name="enc_counts_per_rev"></param>
+            </hardware>
+            <joint name = "left_wheel_joint">
+                <command_interface name = "velocity">
+                    <param name="min">-10.0</param>
+                    <param name="max">10.0</param>
+                </command_interface>
+                <state_interface name = "velocity"/>
+                <state_interface name = "position"/>
+            </joint>
+            <joint name = "right_wheel_joint">
+                <command_interface name = "velocity">
+                    <param name="min">-10.0</param>
+                    <param name="max">10.0</param>
+                </command_interface>
+                <state_interface name = "velocity"/>
+                <state_interface name = "position"/>
+            </joint>
+        </ros2_control>
+    </xacro:unless>
+    <!-- 1B. Simulation mode-->
+    <xacro:if value="$(arg sim_mode)">
+        <ros2_control name="GazeboSystem" type="system">
+            <hardware>
+                <plugin>gazebo_ros2_control/GazeboSystem</plugin>
+            </hardware>
+            <joint name = "left_wheel_joint">
+                <command_interface name = "velocity">
+                    <param name="min">-10.0</param>
+                    <param name="max">10.0</param>
+                </command_interface>
+                <state_interface name = "velocity"/>
+                <state_interface name = "position"/>
+            </joint>
+            <joint name = "right_wheel_joint">
+                <command_interface name = "velocity">
+                    <param name="min">-10.0</param>
+                    <param name="max">10.0</param>
+                </command_interface>
+                <state_interface name = "velocity"/>
+                <state_interface name = "position"/>
+            </joint>
+        </ros2_control>
+    </xacro:if>
     <!-- 2. Introduces the gazebo (simulation) controls-->
     <gazebo>
         <plugin name="gazebo_ros2_control" filename="libgazebo_ros2_control.so">
             <parameters>${find my_bot}/config/my_controllers.yaml</parameters>
+            <parameters>${find my_bot}/config/gaz_ros2_ctl_use_sim.yaml</parameters>
         </plugin>
     </gazebo>
