Commit message: Introducing controller control

File: description/camera.xacro (robot description, xacro)
@@ -6,5 +6,5 @@
         <parent link="chassis"/>
         <child link="camera_link"/>
-        <origin xyz="0.305 0 0.08" rpy="0 0 0"/>
+        <origin xyz="0.305 0 0.08" rpy="0 0.18 0"/>
     </joint>
     <link name="camera_link">

File: description/robot_core.xacro (robot description, xacro)
@@ -34,9 +34,18 @@
         <color rgba="0 0 0 1"/>
     </material>
-    <!-- 4. Defines all the relevant links of the body [Source 3 and 19]-->
-    <!-- 4A. This is the base link, located at the centre of the body. All points will be based of this-->
+    <!-- 4. Introduces the base link and base footprint link-->
+    <!-- 4A. This is the base link, located at the centre of the body. All points will be based of this [Source 3]-->
     <link name="base_link">
     </link>
-    <!-- 4B. This is the chassis, a box with a size of 30cm x 30cm x 15cm, located at the origin of the base link with an x-offset of 15cm and z-offset of 7.5cm-->
+    <!-- 4B. This is the base footprint link [Source 23]-->
+    <joint name="base_footprint_joint" type="fixed">
+        <parent link="base_link"/>
+        <child link="base_footprint"/>
+        <origin xyz="0 0 0"/>
+    </joint>
+    <link name="base_footprint">
+    </link>
+    <!-- 5. Defines all the relevant links of the body [Source 3 and 19]-->
+    <!-- 5A. This is the chassis, a box with a size of 30cm x 30cm x 15cm, located at the origin of the base link with an x-offset of 15cm and z-offset of 7.5cm-->
     <joint name="chassis_joint" type="fixed">
         <parent link="base_link"/>
@@ -65,5 +74,5 @@
         <material>Gazebo/White</material>
     </gazebo>
-    <!-- 3C. This is the left wheel, a cylinder with a radius of 5cm and length of 4cm, with an y-offset of 175mm and rotated 270 degrees around the x-axis-->
+    <!-- 5B. This is the left wheel, a cylinder with a radius of 5cm and length of 4cm, with an y-offset of 175mm and rotated 270 degrees around the x-axis-->
     <joint name="left_wheel_joint" type="continous">
         <parent link="base_link"/>
@@ -91,5 +100,5 @@
         <material>Gazebo/Black</material>
     </gazebo>
-    <!-- 3D. This is the right wheel, a cylinder with a radius of 5cm and length of 4cm, with an y-offset of 175mm and rotated 90 degrees around the x-axis-->
+    <!-- 5C. This is the right wheel, a cylinder with a radius of 5cm and length of 4cm, with an y-offset of 175mm and rotated 90 degrees around the x-axis-->
     <joint name="right_wheel_joint" type="continous">
         <parent link="base_link"/>
@@ -117,5 +126,5 @@
         <material>Gazebo/Black</material>
     </gazebo>
-    <!-- 3E. This is the caster wheel, a sphere with a radius of 5cm, located at an x-offset of 24cm from the chassis-->
+    <!-- 5D. This is the caster wheel, a sphere with a radius of 5cm, located at an x-offset of 24cm from the chassis-->
     <joint name="caster_wheel_joint" type="fixed">
         <parent link="chassis"/>

Commit message: Debugging on several files

File: description/camera.xacro (robot description, xacro)
@@ -1,4 +1,4 @@
 <?xml version="1.0"?>
-<robot xmlns:xacro="http://www.ros.org/wiki/xacro">
+<robot xmlns:xacro="http://www.ros.org/wiki/xacro" name="robot">
     <!-- 1. Creates a joint between lidar and robot body [Source 14]-->
     <!-- 1A. The Camera itself-->
@@ -6,14 +6,14 @@
         <parent link="chassis"/>
         <child link="camera_link"/>
-        <origin xyz="0.305 0 0.08" rpy="0 0.18 0"/>
+        <origin xyz="0.36 0 0.12" rpy="0 0 0"/>
     </joint>
     <link name="camera_link">
         <visual>
             <geometry>
-                <box size="0.01 .03 .03"/>
+                <box size="0.01 0.03 0.03"/>
             </geometry>
             <material name="red"/>
         </visual>
-        <collision>
+        <!--<collision>
             <origin xyz="0.305 0 0.08" rpy="0 0 0"/>
             <geometry>
@@ -23,8 +23,8 @@
         <xacro:inertial_box mass="0.5" x="0.01" y="0.3" z="0.3"/>
             <origin xyz="0.305 0 0.08" rpy="0 0 0"/>
-        </xacro:inertial_box>
+        </xacro:inertial_box>-->
     </link>
     <!-- 1B. The camera optics (an alias to process the different axis than of ROS2)-->
-    <joint name="camera_joint" type="fixed">
+    <joint name="camera_optical_joint" type="fixed">
         <parent link="camera_link"/>
         <child link="camera_link_optical"/>

File: description/gazebo_control.xacro (robot description, xacro)
@@ -4,5 +4,5 @@
     <!-- 1. Introduces the gazebo (simulation) controls-->
     <gazebo>
-        <plugin name="diff_drive" filename="libgazebo_ros_diff_drive.so">
+        <plugin name='diff_drive' filename='libgazebo_ros_diff_drive.so'>
             <!-- 1A. Wheel Details -->
             <left_joint>left_wheel_joint</left_joint>
@@ -12,5 +12,5 @@
             <!-- 1B. The maximum limits-->
             <max_wheel_torque>200</max_wheel_torque>
-            <max_wheel_acceleration>10</max_wheel_acceleration>
+            <max_wheel_acceleration>10.0</max_wheel_acceleration>
             <!-- 1C. Output details-->
             <odometry_frame>odom</odometry_frame>

File: description/lidar.xacro (robot description, xacro)
@@ -1,4 +1,4 @@
 <?xml version="1.0"?>
-<robot xmlns:xacro="http://www.ros.org/wiki/xacro">
+<robot xmlns:xacro="http://www.ros.org/wiki/xacro" name="robot">
     <!-- 1. Creates a joint between lidar and robot body [Source 11]-->
     <joint name="laser_joint" type="fixed">
@@ -8,19 +8,19 @@
     </joint>
     <link name="laser_frame">
-        <visual>
-            <geometry>
-                <cylinder radius="0.05" length="0.04"/>
-            </geometry>
-            <material name="red"/>
-        </visual>
-        <collision>
-            <geometry>
-                <cylinder radius="0.05" length="0.04"/>
-            </geometry>
-        </collision>
-        <xacro:inertial_cylinder mass="0.1" length="0.04" radius="0.05"/>
-            <origin xyz="0 0 0" rpy="-${pi/2} 0 0"/>
-        </xacro:inertial_cylinder>
-    </link>
+    <visual>
+        <geometry>
+            <cylinder radius="0.05" length="0.04"/>
+        </geometry>
+        <material name="red"/>
+    </visual>
+    <collision>
+        <geometry>
+            <cylinder radius="0.05" length="0.04"/>
+        </geometry>
+    </collision>
+    <xacro:inertial_cylinder mass="0.1" length="0.04" radius="0.05">
+        <origin xyz="0 0 0" rpy="0 0 0"/>
+    </xacro:inertial_cylinder>
+</link>
     <!-- 1A. Gazebo reference for laser_frame [Source 12]-->
     <gazebo reference="laser_frame">

File: description/robot_core.xacro (robot description, xacro)
@@ -3,5 +3,5 @@
     <!-- 1. Calls the inertial macros to provide inertia [Source 4]-->
     <xacro:include filename="inertial_macros.xacro"/>
-    <!-- 2. Defines all the relevant dimensions [Source 19]-->
+    <!-- 2. Defines all the relevant dimensions [Source 19]>
     <xacro:property name="chassis_length" value="0.335"/>
     <xacro:property name="chassis_width" value="0.265"/>
@@ -17,6 +17,6 @@
     <xacro:property name="caster_wheel_mass" value="0.01"/>
     <xacro:property name="caster_wheel_offset_x" value="0.075"/>
-    <xacro:property name="caster_wheel_offset_z" value="${wheel_offset_z - wheel_radius + caster_wheel_radius}"/>
-    <!-- 3. Defines all the relevant colours of materials [Source 3]-->
+    <xacro:property name="caster_wheel_offset_z" value="${wheel_offset_z - wheel_radius + caster_wheel_radius}"/>-->
+    <!-- 2. Defines all the relevant colours of materials [Source 3]-->
     <material name="white">
         <color rgba="1 1 1 1"/>
@@ -38,5 +38,5 @@
     <link name="base_link">
     </link>
-    <!-- 4B. This is the base footprint link [Source 23]-->
+    <!-- 4B. This is the base footprint link [Source 23]
     <joint name="base_footprint_joint" type="fixed">
         <parent link="base_link"/>
@@ -45,28 +45,28 @@
     </joint>
     <link name="base_footprint">
-    </link>
+    </link>-->
     <!-- 5. Defines all the relevant links of the body [Source 3 and 19]-->
     <!-- 5A. This is the chassis, a box with a size of 30cm x 30cm x 15cm, located at the origin of the base link with an x-offset of 15cm and z-offset of 7.5cm-->
-    <joint name="chassis_joint" type="fixed">
+     <joint name="chassis_joint" type="fixed">
         <parent link="base_link"/>
         <child link="chassis"/>
-        <origin xyz="${-wheel_offset_x} 0 ${-wheel_offset_z}"/>
+        <origin xyz="-0.1 0 0"/>
     </joint>
     <link name="chassis">
         <visual>
-            <origin xyz="${chassis_length/2} 0 ${chassis_height/2}"/>
+            <origin xyz="0.15 0 0.075" rpy="0 0 0"/>
             <geometry>
-                <box size="${chassis_length} ${chassis_width} ${chassis_height}"/>
+                <box size="0.413 0.286 0.171"/>
             </geometry>
             <material name="white"/>
         </visual>
         <collision>
-            <origin xyz="${chassis_length/2} 0 ${chassis_height/2}"/>
+            <origin xyz="0.15 0 0.075" rpy="0 0 0"/>
             <geometry>
-                <box size="${chassis_length} ${chassis_width} ${chassis_height}"/>
+                <box size="0.413 0.286 0.171"/>
             </geometry>
         </collision>
-        <xacro:inertial_box mass="0.5" x="${chassis_length}" y="${chassis_width}" z="${chassis_height}">
-            <origin xyz="${chassis_length/2} 0 ${chassis_height/2}" rpy="0 0 0"/>
+        <xacro:inertial_box mass="0.5" x="0.3" y="0.3" z="0.15">
+            <origin xyz="0.15 0 0.075" rpy="0 0 0"/>
         </xacro:inertial_box>
     </link>
@@ -75,8 +75,8 @@
     </gazebo>
     <!-- 5B. This is the left wheel, a cylinder with a radius of 5cm and length of 4cm, with an y-offset of 175mm and rotated 270 degrees around the x-axis-->
-    <joint name="left_wheel_joint" type="continous">
+    <joint name="left_wheel_joint" type="continuous">
         <parent link="base_link"/>
         <child link="left_wheel"/>
-        <origin xyz="0 ${wheel_offset_y} 0" rpy="-${pi/2} 0 0" />
+        <origin xyz="0 0.175 0" rpy="-${pi/2} 0 0"/>
         <axis xyz="0 0 1"/>
     </joint>
@@ -84,5 +84,56 @@
         <visual>
             <geometry>
-                <cylinder radius="${wheel_radius}" length="${wheel_thickness}"/>
+                <cylinder radius="0.05" length="0.04"/>
+            </geometry>
+            <material name="blue"/>
+        </visual>
+        <collision>
+            <geometry>
+                <cylinder radius="0.05" length="0.04"/>
+            </geometry>
+        </collision>
+        <xacro:inertial_cylinder mass="0.1" length="0.05" radius="0.05">
+            <origin xyz="0 0 0" rpy="0 0 0"/>
+        </xacro:inertial_cylinder>
+    </link>
+    <gazebo reference="left_wheel">
+        <material>Gazebo/Blue</material>
+    </gazebo>
+    <!-- 5C. This is the right wheel, a cylinder with a radius of 5cm and length of 4cm, with an y-offset of 175mm and rotated 90 degrees around the x-axis-->
+    <joint name="right_wheel_joint" type="continuous">
+        <parent link="base_link"/>
+        <child link="right_wheel"/>
+        <origin xyz="0 -0.175 0" rpy="${pi/2} 0 0"/>
+        <axis xyz="0 0 -1"/>
+    </joint>
+    <link name="right_wheel">
+        <visual>
+            <geometry>
+                <cylinder radius="0.05" length="0.04"/>
+            </geometry>
+            <material name="blue"/>
+        </visual>
+        <collision>
+            <geometry>
+                <cylinder radius="0.05" length="0.04"/>
+            </geometry>
+        </collision>
+        <xacro:inertial_cylinder mass="0.1" length="0.04" radius="0.05">
+            <origin xyz="0 0 0" rpy="0 0 0"/>
+        </xacro:inertial_cylinder>
+    </link>
+    <gazebo reference="right_wheel">
+        <material>Gazebo/Blue</material>
+    </gazebo>
+    <!-- 5D. This is the caster wheel, a sphere with a radius of 5cm, located at an x-offset of 24cm from the chassis-->
+    <joint name="caster_wheel_joint" type="fixed">
+        <parent link="chassis"/>
+        <child link="caster_wheel"/>
+        <origin xyz="0.26 0 0" rpy="0 0 0"/>
+    </joint>
+    <link name="caster_wheel">
+        <visual>
+            <geometry>
+                <sphere radius="0.05" />
             </geometry>
             <material name="black"/>
@@ -90,60 +141,10 @@
         <collision>
             <geometry>
-                <sphere radius="${wheel_radius}"/>
-            </geometry>
-        </collision>
-        <xacro:inertial_cylinder mass="${wheel_mass}" length="${wheel_thickness}" radius="${wheel_radius}">
-            <origin xyz="0 0 0" rpy="-${pi/2} 0 0"/>
-        </xacro:inertial_cylinder>
-    </link>
-    <gazebo reference="left_wheel">
-        <material>Gazebo/Black</material>
-    </gazebo>
-    <!-- 5C. This is the right wheel, a cylinder with a radius of 5cm and length of 4cm, with an y-offset of 175mm and rotated 90 degrees around the x-axis-->
-    <joint name="right_wheel_joint" type="continous">
-        <parent link="base_link"/>
-        <child link="right_wheel"/>
-        <origin xyz="0 ${-wheel_offset_y} 0" rpy="${pi/2} 0 0" />
-        <axis xyz="0 0 -1"/>
-    </joint>
-    <link name="right_wheel">
-        <visual>
-            <geometry>
-                <cylinder radius="${wheel_radius}" length="${wheel_thickness}"/>
+                <sphere radius="0.05" />
             </geometry>
             <material name="black"/>
-        </visual>
-        <collision>
-            <geometry>
-                <sphere radius="${wheel_radius}"/>
-            </geometry>
         </collision>
-        <xacro:inertial_cylinder mass="${wheel_mass}" length="${wheel_thickness}" radius="${wheel_radius}">
-            <origin xyz="0 0 0" rpy="-${pi/2} 0 0"/>
-        </xacro:inertial_cylinder>
-    </link>
-    <gazebo reference="right_wheel">
-        <material>Gazebo/Black</material>
-    </gazebo>
-    <!-- 5D. This is the caster wheel, a sphere with a radius of 5cm, located at an x-offset of 24cm from the chassis-->
-    <joint name="caster_wheel_joint" type="fixed">
-        <parent link="chassis"/>
-        <child link="caster_wheel"/>
-        <origin xyz="${caster_wheel_offset_x} 0 ${caster_wheel_offset_z}"/>
-    </joint>
-    <link name="caster_wheel">
-        <visual>
-            <geometry>
-                <sphere radius="${caster_wheel_radius}"/>
-            </geometry>
-            <material name="black"/>
-        </visual>
-        <collision>
-            <geometry>
-                <sphere radius="${caster_wheel_radius}"/>
-            </geometry>
-        </collision>
-         <xacro:inertial_sphere mass="${caster_wheel_mass}" radius="${caster_wheel_radius}">
-            <origin xyz="0 0 0" rpy ="0 0 0"/>
+        <xacro:inertial_sphere mass="0.1" radius="0.05">
+            <origin xyz="0 0 0" rpy="0 0 0"/>
         </xacro:inertial_sphere>
     </link>
